File: EagleFiles/arduino.brd (EAGLE design)
At the start: 67.9 x 66 mm, 41 parts, among them IC1 4067D, IC2 4067D, IC3 4067D, J1 AVR_SPI, U1 ATMEGA168

Commit message: finally did board layout
now to fix all the errors :(
Parts:
- moved C12 4.00 mm to (30.2, 30.8)
- moved C1 1.00 mm to (45.1, 27.4)
- moved C4 1.00 mm to (21.4, 17.2)
Routing:
- net VCC: track 157.3 -> 241.9 mm, vias 2 -> 9
- net N$43: track 0.00 -> 80.0 mm, vias 0 -> 11
- net N$42: track 0.00 -> 65.1 mm, vias 0 -> 6
- net GND: track 221.9 -> 273.3 mm, vias 4 -> 12
- net N$3: track 75.5 -> 122.5 mm, vias 2 -> 6
- net N$2: track 59.4 -> 104.3 mm, vias 3 -> 10
- net N$81: track 0.00 -> 44.5 mm, vias 0 -> 6
- net N$7: track 63.8 -> 104.7 mm, vias 4 -> 7
- net N$64: track 0.00 -> 40.5 mm, vias 0 -> 6
- net N$75: track 0.00 -> 39.8 mm, vias 0 -> 2
- net N$41: track 25.3 -> 59.3 mm, vias 2 -> 7
- net N$63: track 0.00 -> 33.5 mm, vias 0 -> 4
- net N$23: track 0.00 -> 30.0 mm, vias 0 -> 2
- net N$15: track 0.00 -> 25.5 mm, vias 0 -> 1
- net N$68: track 0.00 -> 25.1 mm, vias 0 -> 2
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